File: SIMO_Non_inverted_Buck_Boost.kicad_pcb (KiCad board)
At the start: 2 copper layers, 218.4 x 92.7 mm, 110 parts, among them J1 Vin1, J101 Vin1_MOS_C, J111 V1AC_MOS_C, J112 V1_AC, J121 V1AC_sens, J2 Vin2, J201 Vin2_MOS_C, J211 V2AC_MOS_C, J212 V2_AC, J221 V2AC_sens, J3 3.3V_rail, J311 V3DC_MOS_C, J312 V3_DC, J321 V3DC_sens, J4 12V_rail, J401 Flywheel_Vin_C, J501 Flywheel_Vout_C, J601 IL_sense, Q101 IPA083N10N5, Q111 IPA083N10N5, Q112 IPA083N10N5, Q202 IPA083N10N5, Q211 IPA083N10N5, Q212 IPA083N10N5, Q311 IPA083N10N5, Q312 IPA083N10N5, Q401 IPA083N10N5, Q402 IPA083N10N5, Q501 IPA083N10N5, Q502 IPA083N10N5, U101 SI8261BAC-C-IS, U111 SI8261BAC-C-IS, U201 SI8261BAC-C-IS, U211 SI8261BAC-C-IS, U311 SI8261BAC-C-IS, U401 SI8261BAC-C-IS, U501 SI8261BAC-C-IS, U601 INA240A4-Q1

Commit message: remove backup file
Parts:
- added REF**: MountingHole_3.5mm, MountingHole:MountingHole_2.7mm_M2.5, F.Cu at (272.4, 116.2)
- added REF**: MountingHole_3.5mm, MountingHole:MountingHole_2.7mm_M2.5, F.Cu at (60.3, 116.2)
- added REF**: MountingHole_3.5mm, MountingHole:MountingHole_2.7mm_M2.5, F.Cu at (60.3, 29.8)
- added REF**: MountingHole_3.5mm, MountingHole:MountingHole_2.7mm_M2.5, F.Cu at (272.4, 29.8)
Changed lines of the file:
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@@
     )
   )
+  (footprint "MountingHole:MountingHole_2.7mm_M2.5" (layer "F.Cu")
+    (at 272.415 116.205)
+    (descr "Mounting Hole 2.7mm, no annular, M2.5")
+    (tags "mounting hole 2.7mm no annular m2.5")
+    (attr exclude_from_pos_files exclude_from_bom)
+    (fp_text reference "REF**" (at 0 -3.7) (layer "F.SilkS") hide
+      (effects (font (size 1 1) (thickness 0.15)))
+    )
+    (fp_text value "MountingHole_3.5mm" (at 0 3.7) (layer "F.Fab")
+      (effects (font (size 1 1) (thickness 0.15)))
+    )
+    (fp_text user "${REFERENCE}" (at 0 0) (layer "F.Fab")
+      (effects (font (size 1 1) (thickness 0.15)))
+    )
+    (fp_circle (center 0 0) (end 2.7 0) (layer "Cmts.User") (width 0.15) (fill none))
+    (fp_circle (center 0 0) (end 2.95 0) (layer "F.CrtYd") (width 0.05) (fill none))
+    (pad "" np_thru_hole circle (at 0 0) (size 2.7 2.7) (drill 2.7) (layers F&B.Cu *.Mask))
+  )
   (footprint "Capacitor_SMD:C_0805_2012Metric_Pad1.18x1.45mm_HandSolder" (layer "F.Cu")
     (at 193.04 87.63)
@@
     )
   )
+  (footprint "MountingHole:MountingHole_2.7mm_M2.5" (layer "F.Cu")
+    (at 60.325 116.205)
+    (descr "Mounting Hole 2.7mm, no annular, M2.5")
+    (tags "mounting hole 2.7mm no annular m2.5")
+    (attr exclude_from_pos_files exclude_from_bom)
+    (fp_text reference "REF**" (at 0 -3.7) (layer "F.SilkS") hide
+      (effects (font (size 1 1) (thickness 0.15)))
+    )
+    (fp_text value "MountingHole_3.5mm" (at 0 3.7) (layer "F.Fab")
+      (effects (font (size 1 1) (thickness 0.15)))
+    )
+    (fp_text user "${REFERENCE}" (at 0 0) (layer "F.Fab")
+      (effects (font (size 1 1) (thickness 0.15)))
+    )
+    (fp_circle (center 0 0) (end 2.7 0) (layer "Cmts.User") (width 0.15) (fill none))
+    (fp_circle (center 0 0) (end 2.95 0) (layer "F.CrtYd") (width 0.05) (fill none))
+    (pad "" np_thru_hole circle (at 0 0) (size 2.7 2.7) (drill 2.7) (layers F&B.Cu *.Mask))
+  )
   (footprint "SIMO_PCB_Lib:SI8261BAC-C-IS" (layer "F.Cu")
     (at 66.04 63.074827 90)
@@
       (net 34 "/V3MOS_S") (pinfunction "S") (pintype "passive"))
   )
+  (footprint "MountingHole:MountingHole_2.7mm_M2.5" (layer "F.Cu")
+    (at 60.325 29.845)
+    (descr "Mounting Hole 2.7mm, no annular, M2.5")
+    (tags "mounting hole 2.7mm no annular m2.5")
+    (attr exclude_from_pos_files exclude_from_bom)
+    (fp_text reference "REF**" (at 0 -3.7) (layer "F.SilkS") hide
+      (effects (font (size 1 1) (thickness 0.15)))
+    )
+    (fp_text value "MountingHole_3.5mm" (at 0 3.7) (layer "F.Fab")
+      (effects (font (size 1 1) (thickness 0.15)))
+    )
+    (fp_text user "${REFERENCE}" (at 0 0) (layer "F.Fab")
+      (effects (font (size 1 1) (thickness 0.15)))
+    )
+    (fp_circle (center 0 0) (end 2.7 0) (layer "Cmts.User") (width 0.15) (fill none))
+    (fp_circle (center 0 0) (end 2.95 0) (layer "F.CrtYd") (width 0.05) (fill none))
+    (pad "" np_thru_hole circle (at 0 0) (size 2.7 2.7) (drill 2.7) (layers *.Cu *.Mask))
+  )
   (footprint "Resistor_SMD:R_0805_2012Metric_Pad1.20x1.40mm_HandSolder" (layer "F.Cu")
     (at 234.315 102.87 90)
@@
     )
   )
+  (footprint "MountingHole:MountingHole_2.7mm_M2.5" (layer "F.Cu")
+    (at 272.415 29.845)
+    (descr "Mounting Hole 2.7mm, no annular, M2.5")
+    (tags "mounting hole 2.7mm no annular m2.5")
+    (attr exclude_from_pos_files exclude_from_bom)
+    (fp_text reference "REF**" (at 0 -3.7) (layer "F.SilkS") hide
+      (effects (font (size 1 1) (thickness 0.15)))
+    )
+    (fp_text value "MountingHole_3.5mm" (at 0 3.7) (layer "F.Fab")
+      (effects (font (size 1 1) (thickness 0.15)))
+    )
+    (fp_text user "${REFERENCE}" (at 0 0) (layer "F.Fab")
+      (effects (font (size 1 1) (thickness 0.15)))
+    )
+    (fp_circle (center 0 0) (end 2.7 0) (layer "Cmts.User") (width 0.15) (fill none))
+    (fp_circle (center 0 0) (end 2.95 0) (layer "F.CrtYd") (width 0.05) (fill none))
+    (pad "" np_thru_hole circle (at 0 0) (size 2.7 2.7) (drill 2.7) (layers F&B.Cu *.Mask))
+  )
   (footprint "SIMO_PCB_Lib:SI8261BAC-C-IS" (layer "F.Cu")
     (at 266.065 57.085 90)
@@
     (effects (font (size 1 1) (thickness 0.15)))
   )
-  (gr_text "GND | 3.3V\n" (at 120.65 104.775) (layer "F.SilkS")
+  (gr_text "GND | 3.3V\n" (at 120.015 104.775) (layer "F.SilkS")
     (effects (font (size 1 1) (thickness 0.15)))
   )
