File: SIMO_Non_inverted_Buck_Boost.kicad_sch (KiCad schematic)
At the start: 39 parts, among them J1 Vin, J10 V2_AC, J11 V2AC_sense, J12 V2AC_MOS_C, J13 V3_DC, J14 V2AC_sense, J15 V3AC_MOS_C, J16 3.3V_rail, J17 5V_rail, J2 Vin_MOS_C, J3 Flywhell_Vin_C, J4 Flywhell_Vout_C, J5 IL_sense, J7 V1_AC, J8 STM32, J9 V1AC_MOS_C, Q1 IPA083N10N5, Q10 IPA083N10N5, Q11 IPA083N10N5, Q2 IPA083N10N5, Q3 IPA083N10N5, Q4 IPA083N10N5, Q5 IPA083N10N5, Q6 IPA083N10N5, Q7 IPA083N10N5, Q8 IPA083N10N5, Q9 IPA083N10N5

Commit message: SIMO V4 - Change footprint, current&voltage sensor
Parts:
- removed C11: 22u, symbol Device:C
- removed C7, C8, C9: 100n, symbol Device:C
- removed J1: Vin, symbol Connector:Conn_01x02_Female
- removed J10: V2_AC, symbol Connector:Conn_01x02_Male
- removed J11, J14: V2AC_sense, symbol Connector:Conn_01x02_Male
- removed J12: V2AC_MOS_C, symbol Connector:Conn_01x01_Female
- removed J13: V3_DC, symbol Connector:Conn_01x02_Male
- removed J15: V3AC_MOS_C, symbol Connector:Conn_01x01_Female
- removed J16: 3.3V_rail, symbol Connector:Conn_01x02_Male
- removed J17: 5V_rail, symbol Connector:Conn_01x02_Male
- removed J2: Vin_MOS_C, symbol Connector:Conn_01x01_Female
- removed J3: Flywhell_Vin_C, symbol Connector:Conn_01x01_Female
- removed J4: Flywhell_Vout_C, symbol Connector:Conn_01x01_Female
- removed J5: IL_sense, symbol Connector:Conn_01x01_Female
- removed J7: V1_AC, symbol Connector:Conn_01x02_Male
- removed J8: STM32, symbol Connector:Conn_01x02_Male
- removed J9: V1AC_MOS_C, symbol Connector:Conn_01x01_Female
- added C102, C112, C121, C122, C202, C212, C221, C222, C312, C321, C402, C502: 100n, Capacitor_SMD:C_0805_2012Metric_Pad1.18x1.45mm_HandSolder, symbol Device:C
- added D121, D221: DIODE, SIMO_PCB_Lib:D_DO-35_SOD27_P7.62mm_Horizontal_Reverse, symbol pspice:DIODE
- added J1: Vin1, TerminalBlock_MetzConnect:TerminalBlock_MetzConnect_Type073_RT02602HBLU_1x02_P5.08mm_Horizontal, symbol Connector_Generic:Conn_01x02
- added J101: Vin1_MOS_C, Connector_PinHeader_2.54mm:PinHeader_1x02_P2.54mm_Vertical, symbol Connector_Generic:Conn_01x02
- added J111: V1AC_MOS_C, Connector_PinHeader_2.54mm:PinHeader_1x02_P2.54mm_Vertical, symbol Connector_Generic:Conn_01x02
- added J112: V1_AC, TerminalBlock_MetzConnect:TerminalBlock_MetzConnect_Type073_RT02602HBLU_1x02_P5.08mm_Horizontal, symbol Connector_Generic:Conn_01x02
- added J121: V1AC_sens, Connector_PinHeader_2.54mm:PinHeader_1x02_P2.54mm_Vertical, symbol Connector_Generic:Conn_01x02
- added J2: Vin2, TerminalBlock_MetzConnect:TerminalBlock_MetzConnect_Type073_RT02602HBLU_1x02_P5.08mm_Horizontal, symbol Connector_Generic:Conn_01x02
- added J201: Vin2_MOS_C, Connector_PinHeader_2.54mm:PinHeader_1x02_P2.54mm_Vertical, symbol Connector_Generic:Conn_01x02
- added J211: V2AC_MOS_C, Connector_PinHeader_2.54mm:PinHeader_1x02_P2.54mm_Vertical, symbol Connector_Generic:Conn_01x02
- added J212: V2_AC, TerminalBlock_MetzConnect:TerminalBlock_MetzConnect_Type073_RT02602HBLU_1x02_P5.08mm_Horizontal, symbol Connector_Generic:Conn_01x02
- added J221: V2AC_sens, Connector_PinHeader_2.54mm:PinHeader_1x02_P2.54mm_Vertical, symbol Connector_Generic:Conn_01x02
- added J3: 3.3V_rail, TerminalBlock_MetzConnect:TerminalBlock_MetzConnect_Type073_RT02602HBLU_1x02_P5.08mm_Horizontal, symbol Connector_Generic:Conn_01x02
- added J311: V3DC_MOS_C, Connector_PinHeader_2.54mm:PinHeader_1x02_P2.54mm_Vertical, symbol Connector_Generic:Conn_01x02
- added J312: V3_DC, TerminalBlock_MetzConnect:TerminalBlock_MetzConnect_Type073_RT02602HBLU_1x02_P5.08mm_Horizontal, symbol Connector_Generic:Conn_01x02
- added J321: V3DC_sens, Connector_PinHeader_2.54mm:PinHeader_1x02_P2.54mm_Vertical, symbol Connector_Generic:Conn_01x02
- added J4: 12V_rail, TerminalBlock_MetzConnect:TerminalBlock_MetzConnect_Type073_RT02602HBLU_1x02_P5.08mm_Horizontal, symbol Connector_Generic:Conn_01x02
- added J401: Flywheel_Vin_C, Connector_PinHeader_2.54mm:PinHeader_1x02_P2.54mm_Vertical, symbol Connector_Generic:Conn_01x02
- added J501: Flywheel_Vout_C, Connector_PinHeader_2.54mm:PinHeader_1x02_P2.54mm_Vertical, symbol Connector_Generic:Conn_01x02
- added J601: IL_sense, Connector_PinHeader_2.54mm:PinHeader_1x02_P2.54mm_Vertical, symbol Connector_Generic:Conn_01x02
- added PS101, PS111, PS201, PS211, PS311, PS401, PS501: PDSE1-S12-S15-S, SIMO_PCB_Lib:PDSE1-S12-S15-S, symbol SIMO_Symbol:PDSE1-S12-S15-S
- added Q101: IPA083N10N5, SIMO_PCB_Lib:IPA083N10N5, symbol Device:Q_NMOS_GDS
- added R101, R111, R201, R211, R311, R401, R501: 220, Resistor_SMD:R_0805_2012Metric_Pad1.20x1.40mm_HandSolder, symbol Device:R
- added R102, R103, R112, R113, R202, R203, R212, R213, R312, R313, R402, R403, R502, R503: 1R - DNP, Resistor_SMD:R_0805_2012Metric_Pad1.20x1.40mm_HandSolder, symbol Device:R
- added R121, R221, R321: 100k, Resistor_SMD:R_0805_2012Metric_Pad1.20x1.40mm_HandSolder, symbol Device:R
- added R122, R123, R222, R223: 10k, Resistor_SMD:R_0805_2012Metric_Pad1.20x1.40mm_HandSolder, symbol Device:R
- added R322: 6k8, Resistor_SMD:R_0805_2012Metric_Pad1.20x1.40mm_HandSolder, symbol Device:R
- added R404: 0R - DNP, Resistor_SMD:R_0805_2012Metric_Pad1.20x1.40mm_HandSolder, symbol Device:R
- added TP101, TP111, TP112, TP202, TP211, TP212, TP311, TP312, TP401, TP501, TP601: TestPoint, TestPoint:TestPoint_Pad_D1.5mm, symbol Connector:TestPoint
- added TP602, TP603: TestPoint, Connector_PinSocket_2.54mm:PinSocket_1x01_P2.54mm_Vertical, symbol Connector:TestPoint
- added U101, U111, U201, U211, U311, U401, U501: SI8261BAC-C-IS, SIMO_PCB_Lib:SI8261BAC-C-IS, symbol SIMO_Symbol:SI8261BAC-C-IS
- added U601: INA240A4-Q1, SIMO_PCB_Lib:SOIC127P600X175-8N, symbol SIMO_Symbol:INA240A4-Q1
- C111: renamed from C1; footprint (none) -> Capacitor_THT:C_Rect_L18.0mm_W7.0mm_P15.00mm_FKS3_FKP3
- C211: renamed from C3; footprint (none) -> Capacitor_THT:C_Rect_L18.0mm_W7.0mm_P15.00mm_FKS3_FKP3
- C311: renamed from C5; footprint (none) -> Capacitor_THT:C_Rect_L26.5mm_W11.5mm_P22.50mm_MKS4
- C601: renamed from C10; footprint (none) -> Capacitor_SMD:C_0805_2012Metric_Pad1.18x1.45mm_HandSolder
- L111: renamed from L2; footprint (none) -> SIMO_PCB_Lib:SRR1260-120M
- L211: renamed from L3; footprint (none) -> SIMO_PCB_Lib:SRR1260-120M
- L601: renamed from L1; footprint (none) -> Inductor_SMD:L_Wuerth_HCI-1350
- Q111: renamed from Q6; footprint (none) -> SIMO_PCB_Lib:IPA083N10N5
- Q112: renamed from Q7; footprint (none) -> SIMO_PCB_Lib:IPA083N10N5
- Q202: renamed from Q1; footprint (none) -> SIMO_PCB_Lib:IPA083N10N5
- Q211: renamed from Q8; footprint (none) -> SIMO_PCB_Lib:IPA083N10N5
- Q212: renamed from Q9; footprint (none) -> SIMO_PCB_Lib:IPA083N10N5
- Q311: renamed from Q10; footprint (none) -> SIMO_PCB_Lib:IPA083N10N5
- Q312: renamed from Q11; footprint (none) -> SIMO_PCB_Lib:IPA083N10N5
- Q401: renamed from Q3; footprint (none) -> SIMO_PCB_Lib:IPA083N10N5
- Q402: renamed from Q2; footprint (none) -> SIMO_PCB_Lib:IPA083N10N5
- Q501: renamed from Q5; footprint (none) -> SIMO_PCB_Lib:IPA083N10N5
- Q502: renamed from Q4; footprint (none) -> SIMO_PCB_Lib:IPA083N10N5
- R605: renamed from R2; footprint (none) -> Resistor_SMD:R_1206_3216Metric_Pad1.30x1.75mm_HandSolder
Connections:
- net GNDD is gone; now on net GNDA: C601.2
- net +3.3V: now also J3.1 (Pin_1), U601.6 (V+)
- net GNDA: now also C102.2, C112.2, C121.2, C122.2, C202.2, C212.2, C221.2, C222.2, C312.2, C321.2, C402.2, C502.2, J1.2 (Pin_2), J112.2 (Pin_2), J121.1 (Pin_1), J2.2 (Pin_2), J212.2 (Pin_2), J221.1 (Pin_1), J3.2 (Pin_2), J312.2 (Pin_2), J321.1 (Pin_1), J4.2 (Pin_2), J601.1 (Pin_1), PS101.1 (GND), PS111.1 (GND), PS201.1 (GND), PS211.1 (GND), PS311.1 (GND), PS401.1 (GND), PS501.1 (GND), R122.1, R123.1, R222.1, R223.1, R322.1, U601.2 (GND), U601.3 (REF2), U601.4 (GND), U601.7 (REF1)
- net V1_AC: now also D121.1 (K), J112.1 (Pin_1), TP112.1
- net V2_AC: now also D221.1 (K), J212.1 (Pin_1), TP212.1
- net V3_DC: now also J312.1 (Pin_1), R321.2, TP312.1
- net at Q202.2 (D): now also J2.1 (Pin_1)
- net Flywheel_Vin/Gate: no longer names the net of Q401.1 (G)
- net Flywheel_Vin/Gate: now also R404.2; no longer Q402.1 (G)
- net Flywheel_Vin/Source renamed Flywhell_Vin_MOS_S
- net Flywhell_Vin_MOS_S: now also PS401.3 (0V), U401.5 (GND)
- net Flywheel_Vout/Gate renamed Flywhell_Vout_MOS_G
- net Flywhell_Vout_MOS_G: now also R503.2, TP501.1
- net Flywheel_Vout/Source renamed Flywhell_Vout_MOS_S
- net Flywhell_Vout_MOS_S: now also PS501.3 (0V), U501.5 (GND)
- net I_sensor/V+ renamed L_V+
- net L_V+: now also U601.8 (+)
- net I_sensor/V-: no longer names the net of Q111.2 (D), Q211.2 (D), Q311.2 (D), Q501.2 (D)
- net I_sensor/V-: now also TP603.1; no longer R605.2
- net V1AC_MOSFET_DR/Gate renamed V1MOS_G
- net V1MOS_G: now also R113.2, TP111.1
- net V1AC_MOSFET_DR/Source renamed V1MOS_S
- net V1MOS_S: now also PS111.3 (0V), U111.5 (GND)
- net V2AC_MOSFET_DR/Gate renamed V2MOS_G
- net V2MOS_G: now also R213.2, TP211.1
- net V2AC_MOSFET_DR/Source renamed V2MOS_S
- net V2MOS_S: now also PS211.3 (0V), U211.5 (GND)
- net V3DC_MOSFET_DR/Gate renamed V3MOS_G
- net V3MOS_G: now also R313.2, TP311.1
- net V3DC_MOSFET_DR/Source renamed V3MOS_S
- net V3MOS_S: now also PS311.3 (0V), U311.5 (GND)
- net Vin_MOSFET_DR/Gate renamed Vin2_MOS_G
- net Vin2_MOS_G: now also R203.2, TP202.1
- net Vin_MOSFET_DR/Source renamed Vin_MOS_S
- net Vin_MOS_S: now also PS101.3 (0V), PS201.3 (0V), Q101.3 (S), TP601.1, U101.5 (GND), U201.5 (GND)
- new net: C221.1, D221.2 (A), R221.2
- new net: R401.2, U401.2 (Anode)
- new net: J401.2 (Pin_2), U401.3 (Cathode)
- new net: R402.1, U401.6 (Vo), U401.7 (Vo)
- new net: PS401.4 (+VOUT), U401.8 (VDD)
- new net: J501.1 (Pin_1), R501.1
- new net: J501.2 (Pin_2), U501.3 (Cathode)
- new net: R501.2, U501.2 (Anode)
- new net: R201.2, U201.2 (Anode)
- new net: J201.2 (Pin_2), U201.3 (Cathode)
- new net: R202.1, U201.6 (Vo), U201.7 (Vo)
- new net: PS201.4 (+VOUT), U201.8 (VDD)
- new net: R502.2, R503.1
- new net: C122.1, J121.2 (Pin_2), R121.1, R122.2, R123.2
- new net: J401.1 (Pin_1), R401.1
- new net: PS311.4 (+VOUT), U311.8 (VDD)
- new net: R212.1, U211.6 (Vo), U211.7 (Vo)
- new net: R212.2, R213.1
- new net: C222.1, J221.2 (Pin_2), R221.1, R222.2, R223.2
- new net: R101.2, U101.2 (Anode)
- new net: J101.2 (Pin_2), U101.3 (Cathode)
- new net: R102.1, U101.6 (Vo), U101.7 (Vo)
- new net: PS101.4 (+VOUT), U101.8 (VDD)
- new net: C121.1, D121.2 (A), R121.2
- new net: C321.1, J321.2 (Pin_2), R321.1, R322.2
- new net: J111.1 (Pin_1), R111.1
- new net: J111.2 (Pin_2), U111.3 (Cathode)
- new net: R312.2, R313.1
- new net: J311.1 (Pin_1), R311.1
- new net: R311.2, U311.2 (Anode)
- new net: PS501.4 (+VOUT), U501.8 (VDD)
- new net: PS111.4 (+VOUT), U111.8 (VDD)
- new net: R111.2, U111.2 (Anode)
- new net: J311.2 (Pin_2), U311.3 (Cathode)
- new net: J601.2 (Pin_2), U601.5
- new net: R202.2, R203.1
- new net: J201.1 (Pin_1), R201.1
- new net: R402.2, R403.1
- new net: R211.2, U211.2 (Anode)
- new net: J211.2 (Pin_2), U211.3 (Cathode)
- new net: PS211.4 (+VOUT), U211.8 (VDD)
- new net: R112.1, U111.6 (Vo), U111.7 (Vo)
- new net: R112.2, R113.1
- new net: R102.2, R103.1
- new net: J211.1 (Pin_1), R211.1
- new net: J1.1 (Pin_1), Q101.2 (D)
- new net: R502.1, U501.6 (Vo), U501.7 (Vo)
- new net: R312.1, U311.6 (Vo), U311.7 (Vo)
- new net: J101.1 (Pin_1), R101.1
- new net +12V: C102.1, C112.1, C202.1, C212.1, C312.1, C402.1, C502.1, J4.1 (Pin_1), PS101.2 (VIN), PS111.2 (VIN), PS201.2 (VIN), PS211.2 (VIN), PS311.2 (VIN), PS401.2 (VIN), PS501.2 (VIN)
- new net Flywhell_Vin_MOS_G: Q402.1 (G), R403.2, R404.1, TP401.1
- new net L_V-: R605.2, TP602.1, U601.1 (-)
- new net Vin1_MOS_G: Q101.1 (G), R103.2, TP101.1
Other:
- removed sheet Flywheel_Vin
- removed sheet Flywheel_Vout
- removed sheet I_sensor
- removed sheet V1AC_MOSFET_DR
- removed sheet V2AC_MOSFET_DR
- removed sheet V3DC_MOSFET_DR
- removed sheet V_Sensing
- removed sheet Vin_MOSFET_DR
- note added: "1 op amp = 1 caps"
- note added: "12V Rail and decoupling Cap"
- note added: "2R for MOSFET damping 220R for current limiting (12mA)"
- note added: "3.056V = (6.8k*48)/(100k+6.8k) #assume 48V as peak DC"
- note added: "3.238V = (5k*68)/(100k+5k) #assume 68V as peak AC"
- note added: "3V = 200*(5A * 3m ohm)"
- note added: "7 Isolated DCDC input = 7 Caps"
- note added: "<-In"
- note added: "Code # 10x: V1 Mos | 20x: V2 Mos 40x: Flywheel Vin side | 50x: Flywheel Vout side 60x: Inductor current measurement 11x: V1AC MOS | 21x: V2AC MOS | 31x: V3DC MOS 12x: V1AC measure | 22x: V2AC measure | 32x: V3DC measure"
- note added: "Flywhell_Vin Driver circuit"
- note added: "Flywhell_Vout Driver circuit"
- note added: "If source float at 10V, Vout = 12+10V"
- note added: "Inductor current sensing"
- note added: "Isolated DCDC"
- note added: "Out->"
- note added: "Peak V1AC sensing"
- note added: "Peak V2AC sensing"
- note added: "Peak V3DC sensing"
- note added: "SI826xxC: Under voltage lockout <12V (VDD must >=12V to turn on)"
- note added: "Single Inductor Multiple Inputs/Ouputs"
- note added: "V1AC Driver circuit"
- note added: "V2AC Driver circuit"
- note added: "V3DC Driver circuit"
- note added: "Vin1 Driver circuit"
- note added: "Vin2 Driver circuit"
- note added: "pulldown res is must for unity gain"
- note removed: "4 op amp = 4 caps + 1 big cap at power supply"
- moved on the sheet: C111, C211, C311, C601, L111, L211, L601, Q111, Q112, Q202, Q211, Q212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

Commit message: remove backup file
Parts:
- removed C601: 100n, Capacitor_SMD:C_0805_2012Metric_Pad1.18x1.45mm_HandSolder, symbol Device:C
- removed J2: Vin2, TerminalBlock_MetzConnect:TerminalBlock_MetzConnect_Type073_RT02602HBLU_1x02_P5.08mm_Horizontal, symbol Connector_Generic:Conn_01x02
- removed J201: Vin2_MOS_C, Connector_PinHeader_2.54mm:PinHeader_1x02_P2.54mm_Vertical, symbol Connector_Generic:Conn_01x02
- removed J3: 3.3V_rail, TerminalBlock_MetzConnect:TerminalBlock_MetzConnect_Type073_RT02602HBLU_1x02_P5.08mm_Horizontal, symbol Connector_Generic:Conn_01x02
- removed J601: IL_sense, Connector_PinHeader_2.54mm:PinHeader_1x02_P2.54mm_Vertical, symbol Connector_Generic:Conn_01x02
- removed PS201: PDSE1-S12-S15-S, SIMO_PCB_Lib:PDSE1-S12-S15-S, symbol SIMO_Symbol:PDSE1-S12-S15-S
- removed Q202: IPA083N10N5, SIMO_PCB_Lib:IPA083N10N5, symbol Device:Q_NMOS_GDS
- removed R102, R103, R112, R113, R202, R203, R212, R213, R312, R313, R402, R403, R502, R503: 1R - DNP, Resistor_SMD:R_0805_2012Metric_Pad1.20x1.40mm_HandSolder, symbol Device:R
- removed R123, R223: 10k, Resistor_SMD:R_0805_2012Metric_Pad1.20x1.40mm_HandSolder, symbol Device:R
- removed R201: 220, Resistor_SMD:R_0805_2012Metric_Pad1.20x1.40mm_HandSolder, symbol Device:R
- removed R404: 0R - DNP, Resistor_SMD:R_0805_2012Metric_Pad1.20x1.40mm_HandSolder, symbol Device:R
- removed R605: 3m, Resistor_SMD:R_1206_3216Metric_Pad1.30x1.75mm_HandSolder, symbol Device:R
- removed TP202: TestPoint, TestPoint:TestPoint_Pad_D1.5mm, symbol Connector:TestPoint
- removed U201: SI8261BAC-C-IS, SIMO_PCB_Lib:SI8261BAC-C-IS, symbol SIMO_Symbol:SI8261BAC-C-IS
- removed U601: INA240A4-Q1, SIMO_PCB_Lib:SOIC127P600X175-8N, symbol SIMO_Symbol:INA240A4-Q1
- L601: value 6u -> 1u
- R122, R222: value 10k -> 24k9
- R322: value 6k8 -> 30k
Connections:
- net L_V- is gone; now on net L_V+: TP602.1
- net Flywhell_Vin_MOS_G: now also Q401.1 (G), U401.6 (Vo), U401.7 (Vo)
- net Flywhell_Vout_MOS_G: now also U501.6 (Vo), U501.7 (Vo)
- net V1MOS_G: now also U111.6 (Vo), U111.7 (Vo)
- net V2MOS_G: now also U211.6 (Vo), U211.7 (Vo)
- net V3MOS_G: now also U311.6 (Vo), U311.7 (Vo)
- net Vin1_MOS_G: now also U101.6 (Vo), U101.7 (Vo)
Other:
- note added: "2.3V = 10(30k)/(100k+30k) #assume 10V nominal Voltage"
- note added: "2.81V = 14.1*(24.9k)/(124.9k) #assume 14.1V (10V_RMS) as peak AC"
- note added: "Code # 10x: V1 Mos (Sin1) 40x: Flywheel Vin side (Sin2) | 50x: Flywheel Vout side (Sin3) 11x: V1AC MOS (Sout1) | 21x: V2AC MOS (Sout2) | 31x: V3DC MOS (Sout3) 12x: V1AC measure | 22x: V2AC measure | 32x: V3DC measure"
- note added: "Sin1 Driver circuit"
- note added: "Sin2 Driver circuit"
- note added: "Sin3 Driver circuit"
- note added: "Sout1 Driver circuit"
- note added: "Sout2 Driver circuit"
- note added: "Sout3 Driver circuit"
- note removed: "1 op amp = 1 caps"
- note removed: "3.056V = (6.8k*48)/(100k+6.8k) #assume 48V as peak DC"
- note removed: "3.238V = (5k*68)/(100k+5k) #assume 68V as peak AC"
- note removed: "3.3V Rail and decoupling Cap"
- note removed: "3V = 200*(5A * 3m ohm)"
- note removed: "Code # 10x: V1 Mos | 20x: V2 Mos 40x: Flywheel Vin side | 50x: Flywheel Vout side 60x: Inductor current measurement 11x: V1AC MOS | 21x: V2AC MOS | 31x: V3DC MOS 12x: V1AC measure | 22x: V2AC measure | 32x: V3DC measure"
- note removed: "Flywhell_Vin Driver circuit"
- note removed: "Flywhell_Vout Driver circuit"
- note removed: "Inductor current sensing"
- note removed: "V1AC Driver circuit"
- note removed: "V2AC Driver circuit"
- note removed: "V3DC Driver circuit"
- note removed: "Vin1 Driver circuit"
- note removed: "Vin2 Driver circuit"
- note removed: "pulldown res is must for unity gain"
- moved on the sheet: C102, C112, C202, C212, C312, C402, C502, J4, J401, J501, PS401, PS501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
